Commit message: modelo de robot con las dimensiones calibradas
1. el modelo de robot ya presenta las dimensiones correpondientes
pero falta calibrar la parte dimanica para que sea los mas cercano al robot

2. falta el plugin del los sensores de distacia para los senosres tof

File: urdf/robot_core.xacro (robot description, xacro)
@@ -61,5 +61,5 @@
         <parent link="chassis"/>
         <child link="right_wheel"/>
-        <origin xyz="-0.0283 -0.0465 -0.0235" rpy="-${pi/2} 0 0"/>
+        <origin xyz="-0.0283 -0.0465 -0.0235" rpy="${pi/2} 0 0"/>
         <axis xyz="0 0 -1"/>
     </joint>
