Commit message: .

File: urdf/gazebo_control.xacro (robot description, xacro)
@@ -7,9 +7,9 @@
             <left_joint>left_wheel_joint</left_joint>
             <right_joint>right_wheel_joint</right_joint>
-            <wheel_separation>0.35</wheel_separation>
-            <wheel_diameter>0.1</wheel_diameter>
+            <wheel_separation>0.093</wheel_separation>
+            <wheel_diameter>0.028</wheel_diameter>
             <!-- limits -->
-            <max_wheel_torque>200</max_wheel_torque>
-            <max_wheel_acceleration>10.0</max_wheel_acceleration>
+            <max_wheel_torque>0.007</max_wheel_torque>
+            <max_wheel_acceleration>1.0</max_wheel_acceleration>
             <!-- outputs -->
             <odometry_frame>odom</odometry_frame>

File: urdf/robot_core.xacro (robot description, xacro)
@@ -1,6 +1,9 @@
 <?xml version="1.0"?>
 <robot xmlns:xacro="http://www.ros.org/wiki/xacro">
-    <!-- Example link -->
     <xacro:include filename="inertial_macros.xacro"/>
+    <!-- dimension de las piezas de robot -->
+    <xacro:property name="ancho_r" value="0.005" />
+    <xacro:property name="radio_r" value="0.014" />
+    <xacro:property name="radio_e" value="0.01" />
     <!-- Example link -->
     <link name="base_link">
@@ -9,30 +12,30 @@
         <parent link="base_link"/>
         <child link="chassis"/>
-        <origin xyz="-0.1 0 0"/>
+        <origin xyz="0 0 0"/>
     </joint>
     <!-- chassis link -->
     <link name="chassis">
         <visual>
-            <origin xyz="0.15 0 0.075"/>
+            <origin xyz="0.0 0 0.0"/>
             <geometry>
-                <box size="0.3 0.3 0.15"/>
+                <mesh filename="file://$(find proyecto_myrobbie3)/meshes/chassis.dae"/>
             </geometry>
             <material name="white"/>
         </visual>
         <collision>
-            <origin xyz="0.15 0 0.075"/>
+            <origin xyz="0.0 0.0 0.0"/>
             <geometry>
-                <box size="0.3 0.3 0.15"/>
+                <mesh filename="file://$(find proyecto_myrobbie3)/meshes/chassis.dae"/>
             </geometry>
         </collision>
-        <xacro:inertial_box mass="0.5" x="0.3" y="0.3" z="0.15">
-            <origin xyz="0.15 0 0.075" rpy="0 0 0"/>
+        <xacro:inertial_box mass="0.32" x="0.12" y="0.08" z="0.05">
+            <origin xyz="0.0 0.0 0.0" rpy="0.0 0.0 0.0"/>
         </xacro:inertial_box>
     </link>
     <!-- left wheel joint -->
     <joint name="left_wheel_joint" type="continuous">
-        <parent link="base_link"/>
+        <parent link="chassis"/>
         <child link="left_wheel"/>
-        <origin xyz="0 0.175 0" rpy="-${pi/2} 0 0"/>
+        <origin xyz="-0.0283 0.0465 -0.0235" rpy="-${pi/2} 0 0"/>
         <axis xyz="0 0 1"/>
     </joint>
@@ -41,5 +44,5 @@
         <visual>
             <geometry>
-                <cylinder radius="0.05" length="0.04"/>
+                <cylinder radius="${radio_r}" length="${ancho_r}"/>
             </geometry>
             <material name="blue"/>
@@ -47,8 +50,8 @@
         <collision>
             <geometry>
-                <cylinder radius="0.05" length="0.04"/>
+                <cylinder radius="${radio_r}" length="${ancho_r}"/>
             </geometry>
         </collision>
-        <xacro:inertial_cylinder mass="0.1" length="0.04" radius="0.05">
+        <xacro:inertial_cylinder mass="0.04" length="${ancho_r}" radius="${radio_r}">
             <origin xyz="0 0 0" rpy="0 0 0"/>
         </xacro:inertial_cylinder>
@@ -56,7 +59,7 @@
     <!-- right wheel joint -->
     <joint name="right_wheel_joint" type="continuous">
-        <parent link="base_link"/>
+        <parent link="chassis"/>
         <child link="right_wheel"/>
-        <origin xyz="0 -0.175 0" rpy="${pi/2} 0 0"/>
+        <origin xyz="-0.0283 -0.0465 -0.0235" rpy="-${pi/2} 0 0"/>
         <axis xyz="0 0 -1"/>
     </joint>
@@ -65,5 +68,5 @@
         <visual>
             <geometry>
-                <cylinder radius="0.05" length="0.04"/>
+                <cylinder radius="${radio_r}" length="${ancho_r}"/>
             </geometry>
             <material name="blue"/>
@@ -71,8 +74,8 @@
         <collision>
             <geometry>
-                <cylinder radius="0.05" length="0.04"/>
+                <cylinder radius="${radio_r}" length="${ancho_r}"/>
             </geometry>
         </collision>
-        <xacro:inertial_cylinder mass="0.1" length="0.04" radius="0.05">
+        <xacro:inertial_cylinder mass="0.04" length="${ancho_r}" radius="${radio_r}">
             <origin xyz="0 0 0" rpy="0 0 0"/>
         </xacro:inertial_cylinder>
@@ -82,11 +85,11 @@
         <parent link="chassis"/>
         <child link="caster_wheel"/>
-        <origin xyz="0.24 0 0"/>
+        <origin xyz="0.05 0 -0.0275"/>
     </joint>
-    <!-- left wheel link -->
+    <!-- caster wheels -->
     <link name="caster_wheel">
         <visual>
             <geometry>
-                <sphere radius="0.05"/>
+                <sphere radius="${radio_e}"/>
             </geometry>
             <material name="black"/>
@@ -94,8 +97,8 @@
         <collision>
             <geometry>
-                <sphere radius="0.05"/>
+                <sphere radius="${radio_e}"/>
             </geometry>
         </collision>
-        <xacro:inertial_sphere mass="0.1" radius="0.05">
+        <xacro:inertial_sphere mass="0.03" radius="${radio_e}">
             <origin xyz="0 0 0" rpy="0 0 0"/>
         </xacro:inertial_sphere>

Commit message: añadir sensor de lidar 1. documencion de codigo( falta) 2. fata la calibracion dimanica del modelo 3. falta la inclusinon de topico laser a ros2

File: urdf/gazebo_control.xacro (robot description, xacro)
@@ -5,16 +5,26 @@
         <plugin name="diff_drive" filename="libgazebo_ros_diff_drive.so">
             <!-- wheels information -->
+            <!-- Nombre de la articulación izquierda, por defecto es `left_joint` -->
             <left_joint>left_wheel_joint</left_joint>
+              <!-- Nombre de la articulación derecha, por defecto es `right_joint` -->
             <right_joint>right_wheel_joint</right_joint>
+            <!-- La distancia desde el centro de una rueda hasta la otra, en metros, por defecto es 0.34 m -->
             <wheel_separation>0.093</wheel_separation>
+            <!-- Diámetro de las ruedas, en metros, por defecto es 0.15 m -->
             <wheel_diameter>0.028</wheel_diameter>
             <!-- limits -->
+            <!-- Máximo torque que las ruedas pueden producir, en Nm, por defecto es 5 Nm -->
             <max_wheel_torque>0.007</max_wheel_torque>
-            <max_wheel_acceleration>1.0</max_wheel_acceleration>
+            <!-- Aceleración de las ruedas, en rad/s^2, por defecto es 0.0 rad/s^2 -->
+            <max_wheel_acceleration>2.5</max_wheel_acceleration>
             <!-- outputs -->
+            <!-- Marco de referencia de la odometría, por defecto es `odom` -->
             <odometry_frame>odom</odometry_frame>
-            <robot_base_frame>base_link</robot_base_frame>
+            <!-- Marco del robot para calcular la odometría, por defecto es `base_footprint` -->
+            <robot_base_frame>chassis</robot_base_frame>
+            <!-- Establecer en true para publicar transformaciones para la odometría, por defecto es true -->
             <publish_odom>true</publish_odom>
             <publish_odom_tf>true</publish_odom_tf>
+            <!-- Establecer en true para publicar transformaciones para los enlaces de las ruedas, por defecto es false -->
             <publish_wheel_tf>true</publish_wheel_tf>
         </plugin>

File: urdf/robot.urdf.xacro (robot description, xacro)
@@ -6,3 +6,4 @@
     <xacro:include filename="inertial_macros.xacro"/>
     <xacro:include filename="gazebo_control.xacro"/>
+    <xacro:include filename="gazebo_sensor.xacro"/>
 </robot>

File: urdf/robot_core.xacro (robot description, xacro)
@@ -6,5 +6,13 @@
     <xacro:property name="radio_r" value="0.014" />
     <xacro:property name="radio_e" value="0.01" />
-    <!-- Example link -->
+    <!-- link para la odometria -->
+    <link name="base_footprint">
+    </link>
+    <joint name="base_footprint_joint" type="fixed">
+        <parent link="base_link"/>
+        <child link="base_footprint"/>
+        <origin xyz="0 0 0"/>
+    </joint>
+    <!-- base del robot -->
     <link name="base_link">
     </link>
@@ -104,4 +112,28 @@
         </xacro:inertial_sphere>
     </link>
+    <!-- sensor tof -->
+    <link name="laser_frame">
+        <visual>
+            <origin xyz="0.0 0 0.0"/>
+            <geometry>
+                <box size="0.04 0.04 0.02"/>
+            </geometry>
+            <material name="blue"/>
+        </visual>
+        <collision>
+            <origin xyz="0.0 0.0 0.0"/>
+            <geometry>
+                <box size="0.04 0.04 0.02"/>
+            </geometry>
+        </collision>
+        <xacro:inertial_box mass="0.02" x="0.04" y="0.04" z="0.02">
+            <origin xyz="0.0 0.0 0.0" rpy="0.0 0.0 0.0"/>
+        </xacro:inertial_box>
+    </link>
+    <joint name="joint_chassis" type="fixed">
+        <origin xyz="0.0 0.0 0.055" rpy="0.0 0.0 0.0"/>
+        <parent link="chassis"/>
+        <child link="laser_frame"/>
+    </joint>
     <gazebo reference="chassis">
         <material>Gazebo/White</material>
@@ -118,3 +150,6 @@
         <mu2 value = "0.001" />
     </gazebo>
+    <gazebo reference="laser_frame">
+        <material>Gazebo/Blue</material>
+    </gazebo>
 </robot>

Commit message: agregacion de un senosor con plugin tipo rango 1. se utilizo la refencia de como configurar el plugin con la migracion de los tags a ros2. 2. se agrago un sensor con capacidad de tener una vision abierta similar a un sensor TOF 3. falta agrega mas sensores TOF en la aplicacion para que ya este listo el robot gemoelo virtual. 4. es posible crear un macro para duplicar los sensores.

File: urdf/gazebo_control.xacro (robot description, xacro)
@@ -4,8 +4,9 @@
     <gazebo>
         <plugin name="diff_drive" filename="libgazebo_ros_diff_drive.so">
-            <!-- wheels information -->
+            <!-- Replace camelCase elements with camel_case ones -->
+            <update_rate>500</update_rate>
             <!-- Nombre de la articulación izquierda, por defecto es `left_joint` -->
             <left_joint>left_wheel_joint</left_joint>
-              <!-- Nombre de la articulación derecha, por defecto es `right_joint` -->
+            <!-- Nombre de la articulación derecha, por defecto es `right_joint` -->
             <right_joint>right_wheel_joint</right_joint>
             <!-- La distancia desde el centro de una rueda hasta la otra, en metros, por defecto es 0.34 m -->
@@ -13,19 +14,10 @@
             <!-- Diámetro de las ruedas, en metros, por defecto es 0.15 m -->
             <wheel_diameter>0.028</wheel_diameter>
-            <!-- limits -->
+            <!-- Marco de referencia de la odometría, por defecto es `odom` -->
+            <odometry_frame>odom</odometry_frame>
             <!-- Máximo torque que las ruedas pueden producir, en Nm, por defecto es 5 Nm -->
             <max_wheel_torque>0.007</max_wheel_torque>
             <!-- Aceleración de las ruedas, en rad/s^2, por defecto es 0.0 rad/s^2 -->
-            <max_wheel_acceleration>2.5</max_wheel_acceleration>
-            <!-- outputs -->
-            <!-- Marco de referencia de la odometría, por defecto es `odom` -->
-            <odometry_frame>odom</odometry_frame>
-            <!-- Marco del robot para calcular la odometría, por defecto es `base_footprint` -->
-            <robot_base_frame>chassis</robot_base_frame>
-            <!-- Establecer en true para publicar transformaciones para la odometría, por defecto es true -->
-            <publish_odom>true</publish_odom>
-            <publish_odom_tf>true</publish_odom_tf>
-            <!-- Establecer en true para publicar transformaciones para los enlaces de las ruedas, por defecto es false -->
-            <publish_wheel_tf>true</publish_wheel_tf>
+            <max_acceleration>2.5</max_acceleration>
         </plugin>
     </gazebo>

File: urdf/gazebo_sensor.xacro (robot description, xacro)
@@ -2,54 +2,48 @@
 <robot xmlns:xacro="http://www.ros.org/wiki/xacro" >
   <gazebo reference="laser_frame">
-    <sensor type="ray" name="head_sensor">
-      <!-- Posición del sensor en relación al modelo base -->
-      <pose>0 0 0 0 0 0</pose>
-      <!-- Indica si se visualiza o no el sensor -->
-      <visualize>true</visualize>
-      <!-- Tasa de actualización del sensor en Hz -->
-      <update_rate>40</update_rate>
-      <ray>
-        <!-- Configuración del haz de rayos -->
-        <scan>
-          <!-- Configuración horizontal del haz -->
-          <horizontal>
-            <!-- Número de muestras de rayos -->
-            <samples>720</samples>
-            <!-- Resolución angular de los rayos en radianes -->
-            <resolution>1</resolution>
-            <!-- Ángulo mínimo del haz -->
-            <min_angle>-1.570796</min_angle>
-            <!-- Ángulo máximo del haz -->
-            <max_angle>1.570796</max_angle>
-          </horizontal>
-        </scan>
-        <!-- Rango de detección del sensor -->
-        <range>
-          <!-- Distancia mínima detectable -->
-          <min>0.08</min>
-          <!-- Distancia máxima detectable -->
-          <max>0.66</max>
-          <!-- Resolución de la distancia detectable -->
-          <resolution>0.001</resolution>
-        </range>
-        <!-- Configuración del ruido del sensor -->
-        <noise>
-          <!-- Tipo de ruido -->
-          <type>gaussian</type>
-          <!-- Parámetros del ruido basados en especificaciones publicadas para el láser Hokuyo,
-               logrando una precisión de "+-30mm" a una distancia < 10m. Una media de 0.0m y
-               desviación estándar de 0.01m pondrán el 99.7% de las muestras dentro de 0.03m de la lectura real. -->
-          <mean>0.0</mean>
-          <stddev>0.003</stddev>
-        </noise>
-      </ray>
-      <!-- Plugin que controla la simulación del sensor Hokuyo -->
-      <plugin name="gazebo_ros_head_hokuyo_controller" filename="libgazebo_ros_laser.so">
-        <!-- Tópico donde se publican las lecturas del láser -->
-        <topicName>sensor_msgs/LaserScan</topicName>
-        <!-- Marco de referencia asociado al sensor -->
-        <frameName>laser_frame</frameName>
-      </plugin>
-    </sensor>
+    <material>Gazebo/Red</material>
+      <sensor type="ray" name="range_sensor">
+        <visualize>true</visualize>
+        <ray>
+          <scan>
+            <horizontal>
+              <samples>10</samples>
+              <resolution>1</resolution>
+              <min_angle>-0.185</min_angle>
+              <max_angle>0.251</max_angle>
+            </horizontal>
+            <vertical>
+              <samples>10</samples>
+              <resolution>1</resolution>
+              <min_angle>-0.185</min_angle>
+              <max_angle>0.251</max_angle>
+            </vertical>
+          </scan>
+          <range>
+            <min>0.100</min>
+            <max>0.600</max>
+            <resolution>0.003</resolution>
+          </range>
+          <!-- Using gazebo's noise instead of plugin's -->
+          <noise>
+            <type>gaussian</type>
+            <mean>0.0</mean>
+            <stddev>0.003</stddev>
+          </noise>
+        </ray>
+        <!-- Using gazebo's update rate instead of plugin's -->
+        <update_rate>30</update_rate>
+        <plugin name="gazebo_ros_range_controller" filename="libgazebo_ros_ray_sensor.so">
+          <!-- Change namespace and output topic so published topic is /rrbot/laser/scan -->
+          <ros>
+            <namespace>/rrbot</namespace>
+            <remapping>~/out:=range</remapping>
+          </ros>
+          <!-- Set output to sensor_msgs/Range to get same output type as gazebo_ros_range -->
+          <output_type>sensor_msgs/Range</output_type>
+          <!-- <frame_name> ommited, will default to range_link -->
+          <frame_name>laser_frame</frame_name>
+        </plugin>
+      </sensor>
   </gazebo>
 </robot>

File: urdf/robot_core.xacro (robot description, xacro)
@@ -150,6 +150,3 @@
         <mu2 value = "0.001" />
     </gazebo>
-    <gazebo reference="laser_frame">
-        <material>Gazebo/Blue</material>
-    </gazebo>
 </robot>
