Commit message: nodo main para el wall followin 1. inclucion de la librerias del package.xml falta geometry_msgs 2. inclucion de las carpetas nesesaria para la ejecucion de paquete 3. configuracion rviz incluido 4. robot_move_launch spawnea el robot a una orientacion especifica 5. nodo_main_myrobbie3 tiene las medicion de los 2 error para el controlador 6. modified de gazebo_sensor para generar una distribuicion de sensores TOF con un xacro 7. robot_core incluye el xacro para la generar la posiciones de los sensores TOF 8. agregacion de wall dentro de gazebo

File: urdf/gazebo_sensor.xacro (robot description, xacro)
@@ -1,7 +1,28 @@
 <?xml version="1.0"?>
-<robot xmlns:xacro="http://www.ros.org/wiki/xacro" >
-  <gazebo reference="laser_frame">
-    <material>Gazebo/Red</material>
-      <sensor type="ray" name="range_sensor">
+<robot xmlns:xacro="http://www.ros.org/wiki/xacro">
+  <xacro:macro name="pose_sensor" params="name_sensor angle parent_link">
+    <link name="${name_sensor}">
+      <visual name="">
+        <geometry>
+          <box size="0.001 0.01 0.01"/>
+        </geometry>
+        <material name="blue">
+          <color rgba= "0.2 0.2 1 1"/>
+        </material>
+      </visual>
+      <collision>
+        <geometry>
+          <box size="0.001 0.01 0.01"/>
+        </geometry>
+      </collision>
+    </link>
+    <joint name="joint_${name_sensor}" type="fixed">
+      <origin xyz="${0.06*cos(radians(angle))} ${0.06*sin(radians(angle))} 0.0" rpy="0.0 -${radians(7.266)} ${radians(angle)}"/>
+      <parent link="${parent_link}"/>
+      <child link="${name_sensor}"/>
+    </joint>
+    <gazebo reference="${name_sensor}">
+      <material>Gazebo/Blue</material>
+      <sensor type="ray" name="range_${name_sensor}">
         <visualize>true</visualize>
         <ray>
@@ -10,12 +31,12 @@
               <samples>10</samples>
               <resolution>1</resolution>
-              <min_angle>-0.185</min_angle>
-              <max_angle>0.251</max_angle>
+              <min_angle>-${radians(12.5)}</min_angle>
+              <max_angle>${radians(12.5)}</max_angle>
             </horizontal>
             <vertical>
               <samples>10</samples>
               <resolution>1</resolution>
-              <min_angle>-0.185</min_angle>
-              <max_angle>0.251</max_angle>
+              <min_angle>-${radians(12.5)}</min_angle>
+              <max_angle>${radians(12.5)}</max_angle>
             </vertical>
           </scan>
@@ -26,9 +47,9 @@
           </range>
           <!-- Using gazebo's noise instead of plugin's -->
-          <noise>
+          <!-- <noise>
             <type>gaussian</type>
             <mean>0.0</mean>
             <stddev>0.003</stddev>
-          </noise>
+          </noise> -->
         </ray>
         <!-- Using gazebo's update rate instead of plugin's -->
@@ -37,13 +58,15 @@
           <!-- Change namespace and output topic so published topic is /rrbot/laser/scan -->
           <ros>
-            <namespace>/rrbot</namespace>
+            <namespace>/${name_sensor}</namespace>
             <remapping>~/out:=range</remapping>
           </ros>
           <!-- Set output to sensor_msgs/Range to get same output type as gazebo_ros_range -->
           <output_type>sensor_msgs/Range</output_type>
+          <radiation_type>infrared</radiation_type>
           <!-- <frame_name> ommited, will default to range_link -->
-          <frame_name>laser_frame</frame_name>
+          <frame_name>${name_sensor}</frame_name>
         </plugin>
       </sensor>
-  </gazebo>
+    </gazebo>
+  </xacro:macro>
 </robot>

File: urdf/robot_core.xacro (robot description, xacro)
@@ -2,8 +2,11 @@
 <robot xmlns:xacro="http://www.ros.org/wiki/xacro">
     <xacro:include filename="inertial_macros.xacro"/>
+    <xacro:include filename="gazebo_sensor.xacro"/>
     <!-- dimension de las piezas de robot -->
     <xacro:property name="ancho_r" value="0.005" />
     <xacro:property name="radio_r" value="0.014" />
     <xacro:property name="radio_e" value="0.01" />
+    <!-- distribucion de angulos -->
+    <xacro:property name="angle_sensor" value="45" />
     <!-- link para la odometria -->
     <link name="base_footprint">
@@ -117,5 +120,5 @@
             <origin xyz="0.0 0 0.0"/>
             <geometry>
-                <box size="0.04 0.04 0.02"/>
+                <cylinder radius="0.06" length="0.01"/>
             </geometry>
             <material name="blue"/>
@@ -124,16 +127,19 @@
             <origin xyz="0.0 0.0 0.0"/>
             <geometry>
-                <box size="0.04 0.04 0.02"/>
+                <cylinder radius="0.06" length="0.01"/>
             </geometry>
         </collision>
-        <xacro:inertial_box mass="0.02" x="0.04" y="0.04" z="0.02">
-            <origin xyz="0.0 0.0 0.0" rpy="0.0 0.0 0.0"/>
-        </xacro:inertial_box>
     </link>
     <joint name="joint_chassis" type="fixed">
-        <origin xyz="0.0 0.0 0.055" rpy="0.0 0.0 0.0"/>
+        <origin xyz="0.0 0.0 0.055" rpy="0.0 0.0 ${radians(-90)}"/>
         <parent link="chassis"/>
         <child link="laser_frame"/>
     </joint>
+    <xacro:pose_sensor name_sensor="sensor_tof_1" angle="${angle_sensor*(-1 + 0.5)}" parent_link="laser_frame" />
+    <xacro:pose_sensor name_sensor="sensor_tof_2" angle="${angle_sensor*(0 + 0.5)}" parent_link="laser_frame" />
+    <xacro:pose_sensor name_sensor="sensor_tof_3" angle="${angle_sensor*(1 + 0.5)}" parent_link="laser_frame" />
+    <xacro:pose_sensor name_sensor="sensor_tof_4" angle="${angle_sensor*(2 + 0.5)}" parent_link="laser_frame" />
+    <xacro:pose_sensor name_sensor="sensor_tof_5" angle="${angle_sensor*(3 + 0.5)}" parent_link="laser_frame" />
+    <xacro:pose_sensor name_sensor="sensor_tof_6" angle="${angle_sensor*(4 + 0.5)}" parent_link="laser_frame" />
     <gazebo reference="chassis">
         <material>Gazebo/White</material>
@@ -145,4 +151,7 @@
         <material>Gazebo/Blue</material>
     </gazebo>
+    <gazebo reference="laser_frame">
+        <material>Gazebo/Red</material>
+    </gazebo>
     <gazebo reference="caster_wheel">
         <material>Gazebo/Black</material>
